Commit message: Added 2D map generation using navigation stack

File: robot1_description/urdf/robot1_base.xacro (robot description, xacro)
@@ -1,7 +1,7 @@
 <?xml version="1.0"?>
 <robot xmlns:xacro="http://www.ros.org/wiki/xacro"
- 	xmlns:sensor="http://playerstage.sourceforge.net/gazebo/xmlschema/#sensor"
-    	xmlns:controller="http://playerstage.sourceforge.net/gazebo/xmlschema/#controller"
-    	xmlns:interface="http://playerstage.sourceforge.net/gazebo/xmlschema/#interface"
+	xmlns:sensor="http://playerstage.sourceforge.net/gazebo/xmlschema/#sensor"
+	xmlns:controller="http://playerstage.sourceforge.net/gazebo/xmlschema/#controller"
+	xmlns:interface="http://playerstage.sourceforge.net/gazebo/xmlschema/#interface"
 	name="robot1_xacro">
 	<xacro:property name="length_wheel" value="0.05" />
@@ -15,4 +15,5 @@
 		</inertial>
 	</xacro:macro>
+	<xacro:include filename="$(find robot1_description)/urdf/robot.gazebo" />
 	<link name = "base_footprint">
 		<visual>
@@ -24,9 +25,4 @@
 		<xacro:default_inertial mass="0.0001"/>
 	</link>
-	<xacro:include filename="$(find robot1_description)/urdf/robot.gazebo" />
-	<gazebo reference="base_footprint">
-		<material>Gazebo/Green</material>
-		<turnGravityOff>false</turnGravityOff>
-	</gazebo>
 	<link name="base_link">
 		<visual>
@@ -41,8 +37,76 @@
 		<collision>
 			<geometry>
-				<box size="0.2 0.3 0.1"/>
+				<box size="0.2 .3 .1"/>
 			</geometry>
 		</collision>
 		<xacro:default_inertial mass="10"/>
+	</link>
+	<link name="wheel_1">
+		<visual>
+			<geometry>
+				<cylinder length="${length_wheel}" radius="${radius_wheel}"/>
+			</geometry>
+			<origin rpy="0 0 0" xyz="0 0 0"/>
+			<material name="black">
+				<color rgba="0 0 0 1"/>
+			</material>
+		</visual>
+		<collision>
+			<geometry>
+				<cylinder length="${length_wheel}" radius="${radius_wheel}"/>
+			</geometry>
+		</collision>
+		<xacro:default_inertial mass="1"/>
+	</link>
+	<link name="wheel_2">
+		<visual>
+			<geometry>
+				<cylinder length="${length_wheel}" radius="${radius_wheel}"/>
+			</geometry>
+			<origin rpy="0 0 0" xyz="0 0 0"/>
+			<material name="black">
+				<color rgba="0 0 0 1"/>
+			</material>
+		</visual>
+		<collision>
+			<geometry>
+				<cylinder length="${length_wheel}" radius="${radius_wheel}"/>
+			</geometry>
+		</collision>
+		<xacro:default_inertial mass="1"/>
+	</link>
+	<link name="wheel_3">
+		<visual>
+			<geometry>
+				<cylinder length="${length_wheel}" radius="${radius_wheel}"/>
+			</geometry>
+			<origin rpy="0 0 0" xyz="0 0 0"/>
+			<material name="black">
+				<color rgba="0 0 0 1"/>
+			</material>
+		</visual>
+		<collision>
+			<geometry>
+				<cylinder length="${length_wheel}" radius="${radius_wheel}"/>
+			</geometry>
+		</collision>
+		<xacro:default_inertial mass="1"/>
+	</link>
+	<link name="wheel_4">
+		<visual>
+			<geometry>
+				<cylinder length="${length_wheel}" radius="${radius_wheel}"/>
+			</geometry>
+			<origin rpy="0 0 0" xyz="0 0 0"/>
+			<material name="black">
+				<color rgba="0 0 0 1"/>
+			</material>
+		</visual>
+		<collision>
+			<geometry>
+				<cylinder length="${length_wheel}" radius="${radius_wheel}"/>
+			</geometry>
+		</collision>
+		<xacro:default_inertial mass="1"/>
 	</link>
 	<joint name="base_footprint_joint" type="fixed">
@@ -51,76 +115,8 @@
 		<child link="base_link"/>
 	</joint>
-	<link name="wheel_1">
-		<visual>
-			<geometry>
-				<cylinder length="${length_wheel}" radius="${radius_wheel}"/>
-			</geometry>
-			<origin rpy="0 0 0" xyz="0 0 0"/>
-			<material name="black">
-				<color rgba="0 0 0 1"/>
-			</material>
-		</visual>
-		<collision>
-			<geometry>
-				<cylinder length="${length_wheel}" radius="${radius_wheel}"/>
-			</geometry>
-		</collision>
-		<xacro:default_inertial mass="1"/>
-	</link>
-	<link name="wheel_2">
-		<visual>
-			<geometry>
-				<cylinder length="${length_wheel}" radius="${radius_wheel}"/>
-			</geometry>
-			<origin rpy="0 0 0" xyz="0 0 0"/>
-			<material name="black">
-				<color rgba="0 0 0 1"/>
-			</material>
-		</visual>
-		<collision>
-			<geometry>
-				<cylinder length="${length_wheel}" radius="${radius_wheel}"/>
-			</geometry>
-		</collision>
-		<xacro:default_inertial mass="1"/>
-	</link>
-	<link name="wheel_3">
-		<visual>
-			<geometry>
-				<cylinder length="${length_wheel}" radius="${radius_wheel}"/>
-			</geometry>
-			<origin rpy="0 0 0" xyz="0 0 0"/>
-			<material name="black">
-				<color rgba="0 0 0 1"/>
-			</material>
-		</visual>
-		<collision>
-			<geometry>
-				<cylinder length="${length_wheel}" radius="${radius_wheel}"/>
-			</geometry>
-		</collision>
-		<xacro:default_inertial mass="1"/>
-	</link>
-	<link name="wheel_4">
-		<visual>
-			<geometry>
-				<cylinder length="${length_wheel}" radius="${radius_wheel}"/>
-			</geometry>
-			<origin rpy="0 0 0" xyz="0 0 0"/>
-			<material name="black">
-				<color rgba="0 0 0 1"/>
-			</material>
-		</visual>
-		<collision>
-			<geometry>
-				<cylinder length="${length_wheel}" radius="${radius_wheel}"/>
-			</geometry>
-		</collision>
-		<xacro:default_inertial mass="1"/>
-	</link>
 	<joint name="base_to_wheel1" type="continuous">
 		<parent link="base_link"/>
 		<child link="wheel_1"/>
-		<origin rpy="1.5707 0 0" xyz="0.1 0.15 0"/>
+		<origin rpy="-1.5707 0 0" xyz="0.1 0.15 0"/>
 		<axis xyz="0 0 1"/>
 	</joint>
@@ -131,5 +127,5 @@
 		<parent link="base_link"/>
 		<child link="wheel_2"/>
-		<origin rpy="1.5707 0 0" xyz="-0.1 0.15 0"/>
+		<origin rpy="-1.5707 0 0" xyz="-0.1 0.15 0"/>
 	</joint>
 	<joint name="base_to_wheel3" type="continuous">
@@ -137,5 +133,5 @@
 		<child link="wheel_3"/>
 		<axis xyz="0 0 1"/>
-		<origin rpy="1.5707 0 0" xyz="0.1 -0.15 0"/>
+		<origin rpy="-1.5707 0 0" xyz="0.1 -0.15 0"/>
 	</joint>
 	<joint name="base_to_wheel4" type="continuous">
@@ -143,6 +139,7 @@
 		<child link="wheel_4"/>
 		<axis xyz="0 0 1"/>
-		<origin rpy="1.5707 0 0" xyz="-0.1 -0.15 0"/>
-	</joint>
+		<origin rpy="-1.5707 0 0" xyz="-0.1 -0.15 0"/>
+	</joint>
+	<!-- Camera -->
 	<link name="camera_link">
 		<collision>
@@ -173,4 +170,5 @@
 		<child link="camera_link"/>
 	</joint>
+	<!--Hokuyo laser -->
 	<link name="hokuyo_link">
 		<collision>
@@ -198,3 +196,20 @@
 		<child link="hokuyo_link"/>
 	</joint>
+	<!--Drive controller -->
+	<gazebo>
+		<plugin name="skid_steer_driver_controller" 			filename="libgazebo_ros_skid_steer_drive.so">
+			<updateRate>100.0</updateRate>
+			<robotNameSpace>/</robotNameSpace>
+			<leftFrontJoint>base_to_wheel1</leftFrontJoint>
+			<rightFrontJoint>base_to_wheel3</rightFrontJoint>
+			<leftRearJoint>base_to_wheel2</leftRearJoint>
+			<rightRearJoint>base_to_wheel4</rightRearJoint>
+			<wheelSeparation>4</wheelSeparation>
+			<wheelDiameter>0.1</wheelDiameter>
+			<robotBaseFrame>base_link</robotBaseFrame>
+			<torque>1</torque>
+			<topicName>cmd_vel</topicName>
+			<broadcastTF>0</broadcastTF>
+		</plugin>
+	</gazebo>
 </robot>
